Commit message: gazebo done, imu to be fixed

File: robot_description/urdf/bipedal.ros2_control.xacro (robot description, xacro)
@@ -1,8 +1,7 @@
 <?xml version="1.0"?>
 <robot xmlns:xacro="http://www.ros.org/wiki/xacro" name="bipedal">
-    <ros2_control name="bipedal_ros2_control" type="system">
+    <ros2_control name="GazeboSystem" type="system">
         <hardware>
-            <plugin>mock_components/GenericSystem</plugin>
-            <param name="calculate_dynamics">true</param>
+            <plugin>gz_ros2_control/GazeboSimSystem</plugin>
         </hardware>
         <joint name="left_hip_joint">
@@ -30,4 +29,4 @@
             <state_interface name="effort"/>
         </joint>
-    </ros2_control>
+</ros2_control>
 </robot>

File: robot_description/urdf/bipedal.urdf.xacro (robot description, xacro)
@@ -5,4 +5,5 @@
     <xacro:include filename="parts/leg.xacro" />
     <xacro:include filename="bipedal.ros2_control.xacro" />
+    <xacro:include filename="bipedal.gazebo.xacro" />
     <link name="base_footprint"/>
     <joint name="base_link_joint" type="fixed">

File: robot_description/urdf/parts/leg.xacro (robot description, xacro)
@@ -62,5 +62,5 @@
             <visual>
                 <geometry>
-                    <box size="0.15 0.1 0.03"/>
+                    <box size="0.15 0.2 0.03"/>
                 </geometry>
                 <origin xyz="0.05 0 0" rpy="0 0 1.570796"/>
@@ -69,5 +69,5 @@
             <collision>
                 <geometry>
-                    <box size="0.15 0.1 0.03"/>
+                    <box size="0.15 0.2 0.03"/>
                 </geometry>
                  <origin xyz="0.05 0 0" rpy="0 0 1.570796"/>

File: robot_description/urdf/parts/torso.xacro (robot description, xacro)
@@ -24,4 +24,17 @@
             </inertial>
         </link>
+        <gazebo reference="torso">
+            <sensor name="imu_sensor" type="imu">
+                <always_on>true</always_on>
+                <update_rate>100</update_rate>
+                <topic>/bipedal/imu</topic>
+            </sensor>
+        </gazebo>
+        <link name="imu_link"/>
+        <joint name="imu_joint" type="fixed">
+            <parent link="torso"/>
+            <child link="imu_link"/>
+            <origin xyz="0 0 0" rpy="0 0 0"/>
+        </joint>
     </xacro:macro>
 </robot>
