Commit message: started learning

File: robot_description/urdf/bipedal.gazebo.xacro (robot description, xacro)
@@ -73,4 +73,10 @@
         <springReference>0</springReference>
     </gazebo>
+    <!-- ADDED: Gazebo properties for the left ankle joint -->
+    <gazebo reference="left_ankle_joint">
+        <implicitSpringDamper>true</implicitSpringDamper>
+        <springStiffness>0</springStiffness>
+        <springReference>0</springReference>
+    </gazebo>
     <gazebo reference="right_hip_joint">
         <implicitSpringDamper>true</implicitSpringDamper>
@@ -83,3 +89,9 @@
         <springReference>0</springReference>
     </gazebo>
+    <!-- ADDED: Gazebo properties for the right ankle joint -->
+    <gazebo reference="right_ankle_joint">
+        <implicitSpringDamper>true</implicitSpringDamper>
+        <springStiffness>0</springStiffness>
+        <springReference>0</springReference>
+    </gazebo>
 </robot>

File: robot_description/urdf/bipedal.ros2_control.xacro (robot description, xacro)
@@ -17,4 +17,11 @@
             <state_interface name="effort"/>
         </joint>
+        <!-- ADDED: left_ankle_joint definition -->
+        <joint name="left_ankle_joint">
+            <command_interface name="position"/>
+            <state_interface name="position"/>
+            <state_interface name="velocity"/>
+            <state_interface name="effort"/>
+        </joint>
         <joint name="right_hip_joint">
             <command_interface name="position"/>
@@ -29,4 +36,11 @@
             <state_interface name="effort"/>
         </joint>
+        <!-- ADDED: right_ankle_joint definition -->
+        <joint name="right_ankle_joint">
+            <command_interface name="position"/>
+            <state_interface name="position"/>
+            <state_interface name="velocity"/>
+            <state_interface name="effort"/>
+        </joint>
 </ros2_control>
 </robot>

File: robot_description/urdf/bipedal.urdf.xacro (robot description, xacro)
@@ -15,8 +15,8 @@
     <xacro:torso parent="base_link" />
     <xacro:leg prefix="left" parent="torso">
-        <origin xyz="0 0.1 -0.25" rpy="0 0 0"/>
+        <origin xyz="-0.05 0.1 -0.125" rpy="0 0 0"/>
     </xacro:leg>
     <xacro:leg prefix="right" parent="torso">
-        <origin xyz="0 -0.1 -0.25" rpy="0 0 0"/>
+        <origin xyz="-0.05 -0.1 -0.125" rpy="0 0 0"/>
     </xacro:leg>
 </robot>

File: robot_description/urdf/parts/leg.xacro (robot description, xacro)
@@ -12,17 +12,18 @@
             <visual>
                 <geometry>
-                    <cylinder radius="0.05" length="0.4"/>
+                        <cylinder radius="0.05" length="0.2"/>
                 </geometry>
-                <origin xyz="0 0 -0.2" rpy="0 0 0"/>
+                    <origin xyz="0 0 -0.1" rpy="0 0 0"/>
                 <material name="blue"/>
             </visual>
             <collision>
                 <geometry>
-                    <cylinder radius="0.05" length="0.4"/>
+                        <cylinder radius="0.05" length="0.2"/>
                 </geometry>
-                <origin xyz="0 0 -0.2" rpy="0 0 0"/>
+                    <origin xyz="0 0 -0.1" rpy="0 0 0"/>
             </collision>
             <inertial>
-                <mass value="3.5"/>
+                <!-- CHANGE: Reduced mass from 3.5 to 2.0 -->
+                <mass value="4.0"/>
                 <inertia ixx="0.01" ixy="0.0" ixz="0.0" iyy="0.01" iyz="0.0" izz="0.01"/>
             </inertial>
@@ -31,5 +32,5 @@
             <parent link="${prefix}_thigh"/>
             <child link="${prefix}_shin"/>
-            <origin xyz="0 0 -0.4" rpy="0 0 0"/>
+                <origin xyz="0 0 -0.2" rpy="0 0 0"/>
             <axis xyz="0 1 0"/>
             <limit lower="0" upper="1.57" effort="100" velocity="5"/>
@@ -38,44 +39,59 @@
             <visual>
                 <geometry>
-                    <cylinder radius="0.04" length="0.35"/>
+                        <cylinder radius="0.04" length="0.15"/>
                 </geometry>
-                <origin xyz="0 0 -0.175" rpy="0 0 0"/>
+                    <origin xyz="0 0 -0.075" rpy="0 0 0"/>
                 <material name="grey"/>
             </visual>
             <collision>
                 <geometry>
-                    <cylinder radius="0.04" length="0.35"/>
-                </geometry>
-                <origin xyz="0 0 -0.175" rpy="0 0 0"/>
+                        <cylinder radius="0.04" length="0.15"/>
+                </geometry>leg
+                    <origin xyz="0 0 -0.075" rpy="0 0 0"/>
             </collision>
             <inertial>
-                <mass value="1.5"/>
+                <!-- Mass of 1.5 is okay here -->
+                <mass value="3.0"/>
                 <inertia ixx="0.01" ixy="0.0" ixz="0.0" iyy="0.01" iyz="0.0" izz="0.01"/>
             </inertial>
         </link>
-        <joint name="${prefix}_foot_joint" type="fixed">
+        <!-- CRITICAL CHANGE: Replaced fixed joint with a revolute ankle joint -->
+        <joint name="${prefix}_ankle_joint" type="revolute">
             <parent link="${prefix}_shin"/>
             <child link="${prefix}_foot"/>
-            <origin xyz="0 0 -0.35" rpy="0 0 0"/>
+            <origin xyz="0 0 -0.15" rpy="0 0 0"/>
+            <axis xyz="0 1 0"/>
+            <!-- Limit ankle motion to about +/- 30 degrees -->
+            <limit lower="-0.52" upper="0.52" effort="100" velocity="5"/>
         </joint>
         <link name="${prefix}_foot">
             <visual>
                 <geometry>
-                    <box size="0.15 0.2 0.03"/>
+                        <!-- CHANGE: Increased foot length from 0.2 to 0.25 for stability -->
+                        <box size="0.15 0.25 0.015"/>
                 </geometry>
-                <origin xyz="0.05 0 0" rpy="0 0 1.570796"/>
+                    <origin xyz="0.05 0 0" rpy="0 0 1.570796"/>
                 <material name="blue"/>
             </visual>
             <collision>
                 <geometry>
-                    <box size="0.15 0.2 0.03"/>
+                       <!-- CHANGE: Increased foot length from 0.2 to 0.25 for stability -->
+                       <box size="0.15 0.25 0.015"/>
                 </geometry>
-                 <origin xyz="0.05 0 0" rpy="0 0 1.570796"/>
+                     <origin xyz="0.05 0 0" rpy="0 0 1.570796"/>
             </collision>
              <inertial>
-                <mass value="1.5"/>
+                <!-- Mass of 1.5 is okay here -->
+                <mass value="3.5"/>
                 <inertia ixx="0.001" ixy="0.0" ixz="0.0" iyy="0.001" iyz="0.0" izz="0.001"/>
             </inertial>
         </link>
+        <!-- Add a fixed joint for the foot sensor/contact point if needed later -->
+        <joint name="${prefix}_foot_contact_joint" type="fixed">
+          <parent link="${prefix}_foot"/>
+          <child link="${prefix}_foot_contact"/>
+          <origin xyz="0 0 0" rpy="0 0 0"/>
+        </joint>
+        <link name="${prefix}_foot_contact"/>
     </xacro:macro>
 </robot>

File: robot_description/urdf/parts/torso.xacro (robot description, xacro)
@@ -10,5 +10,5 @@
 <visual>
 <geometry>
-<box size="0.25 0.2 0.5"/>
+<box size="0.15 0.2 0.25"/>
 </geometry>
 <material name="grey"/>
@@ -16,9 +16,10 @@
 <collision>
 <geometry>
-<box size="0.25 0.2 0.5"/>
+<box size="0.15 0.2 0.25"/>
 </geometry>
 </collision>
 <inertial>
-<mass value="2.5"/>
+<!-- CHANGE: Increased mass from 2.5 to 6.0 to lower center of mass -->
+<mass value="6.0"/>
 <inertia ixx="0.1" ixy="0.0" ixz="0.0" iyy="0.1" iyz="0.0" izz="0.1"/>
 </inertial>
