Commit message: added rl script, dont know if it works!

File: robot_description/urdf/parts/leg.xacro (robot description, xacro)
@@ -24,5 +24,5 @@
             </collision>
             <inertial>
-                <mass value="1.5"/>
+                <mass value="3.5"/>
                 <inertia ixx="0.01" ixy="0.0" ixz="0.0" iyy="0.01" iyz="0.0" izz="0.01"/>
             </inertial>
@@ -50,5 +50,5 @@
             </collision>
             <inertial>
-                <mass value="1"/>
+                <mass value="1.5"/>
                 <inertia ixx="0.01" ixy="0.0" ixz="0.0" iyy="0.01" iyz="0.0" izz="0.01"/>
             </inertial>
@@ -74,5 +74,5 @@
             </collision>
              <inertial>
-                <mass value="0.5"/>
+                <mass value="1.5"/>
                 <inertia ixx="0.001" ixy="0.0" ixz="0.0" iyy="0.001" iyz="0.0" izz="0.001"/>
             </inertial>

File: robot_description/urdf/parts/torso.xacro (robot description, xacro)
@@ -1,40 +1,83 @@
 <?xml version="1.0"?>
 <robot xmlns:xacro="http://www.ros.org/wiki/xacro">
-    <xacro:macro name="torso" params="parent">
-        <joint name="torso_joint" type="fixed">
-            <parent link="${parent}"/>
-            <child link="torso"/>
-            <origin xyz="0 0 0.5" rpy="0 0 0"/>
-        </joint>
-        <link name="torso">
-            <visual>
-                <geometry>
-                    <box size="0.25 0.2 0.5"/>
-                </geometry>
-                <material name="grey"/>
-            </visual>
-            <collision>
-                <geometry>
-                    <box size="0.25 0.2 0.5"/>
-                </geometry>
-            </collision>
-            <inertial>
-                <mass value="5"/>
-                <inertia ixx="0.1" ixy="0.0" ixz="0.0" iyy="0.1" iyz="0.0" izz="0.1"/>
-            </inertial>
-        </link>
-        <gazebo reference="torso">
-            <sensor name="imu_sensor" type="imu">
-                <always_on>true</always_on>
-                <update_rate>100</update_rate>
-                <topic>/bipedal/imu</topic>
-            </sensor>
-        </gazebo>
-        <link name="imu_link"/>
-        <joint name="imu_joint" type="fixed">
-            <parent link="torso"/>
-            <child link="imu_link"/>
-            <origin xyz="0 0 0" rpy="0 0 0"/>
-        </joint>
-    </xacro:macro>
+<xacro:macro name="torso" params="parent">
+<joint name="torso_joint" type="fixed">
+<parent link="${parent}"/>
+<child link="torso"/>
+<origin xyz="0 0 0.5" rpy="0 0 0"/>
+</joint>
+<link name="torso">
+<visual>
+<geometry>
+<box size="0.25 0.2 0.5"/>
+</geometry>
+<material name="grey"/>
+</visual>
+<collision>
+<geometry>
+<box size="0.25 0.2 0.5"/>
+</geometry>
+</collision>
+<inertial>
+<mass value="2.5"/>
+<inertia ixx="0.1" ixy="0.0" ixz="0.0" iyy="0.1" iyz="0.0" izz="0.1"/>
+</inertial>
+</link>
+<gazebo reference="torso">
+<sensor name="imu_sensor" type="imu">
+<always_on>1</always_on>
+<update_rate>100</update_rate>
+<visualize>true</visualize>
+<topic>/bipedal/imu</topic>
+<imu>
+<angular_velocity>
+<x>
+<noise type="gaussian">
+<mean>0.0</mean>
+<stddev>2e-4</stddev>
+</noise>
+</x>
+<y>
+<noise type="gaussian">
+<mean>0.0</mean>
+<stddev>2e-4</stddev>
+</noise>
+</y>
+<z>
+<noise type="gaussian">
+<mean>0.0</mean>
+<stddev>2e-4</stddev>
+</noise>
+</z>
+</angular_velocity>
+<linear_acceleration>
+<x>
+<noise type="gaussian">
+<mean>0.0</mean>
+<stddev>1.7e-2</stddev>
+</noise>
+</x>
+<y>
+<noise type="gaussian">
+<mean>0.0</mean>
+<stddev>1.7e-2</stddev>
+</noise>
+</y>
+<z>
+<noise type="gaussian">
+<mean>0.0</mean>
+<stddev>1.7e-2</stddev>
+</noise>
+</z>
+</linear_acceleration>
+</imu>
+</sensor>
+</gazebo>
+<link name="imu_link"/>
+<joint name="imu_joint" type="fixed">
+<parent link="torso"/>
+<child link="imu_link"/>
+<origin xyz="0 0 0" rpy="0 0 0"/>
+</joint>
+</xacro:macro>
 </robot>
